File: reddit-snoo-meetup.kicad_pcb (KiCad board)
At the start: 2 copper layers, 53.7 x 76 mm, 11 parts, among them X1 Badgelife_sao_connector_v169b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

Commit message: updated gerbers
Parts:
- removed the G*** at (0.00, 0.00) (x5)
- added G*** (x5): LOGO, LOGO, F.Cu at (0.00, 0.00)
Changed lines of the file:
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@@
     (visible_elements 7FFFFFFF)
     (pcbplotparams
-      (layerselection 0x010f0_80000001)
+      (layerselection 0x010f0_ffffffff)
       (usegerberextensions false)
       (usegerberattributes false)
@@
       (outputformat 1)
       (mirror false)
-      (drillshape 1)
+      (drillshape 0)
       (scaleselection 1)
       (outputdirectory "gerbers/"))
@@
     (add_net "Net-(X1-Pad5)")
     (add_net "Net-(X1-Pad6)")
+  )
+  (module my-ki-cad-parts:Badgelife-SAOv169-SAO-2x3 (layer F.Cu)
+    (at 1.4224 29.6164)
+    (descr "Through hole straight IDC box header, 2x03, 2.54mm pitch, double rows")
+    (tags "Through hole IDC box header THT 2x03 2.54mm double row")
+    (fp_text reference X1 (at 0 -5.842) (layer B.SilkS)
+      (effects (font (size 1 1) (thickness 0.15)) (justify mirror))
+    )
+    (fp_text value Badgelife_sao_connector_v169bis (at 0 -7.7) (layer F.Fab)
+      (effects (font (size 1 1) (thickness 0.15)))
+    )
+    (fp_text user %R (at 0.06 0.02 270) (layer F.Fab)
+      (effects (font (size 1 1) (thickness 0.15)))
+    )
+    (fp_line (start -2.54 -4.064) (end -7.366 -4.064) (layer B.SilkS) (width 0.7))
+    (fp_line (start 7.27964 -4.1148) (end 2.54 -4.1148) (layer B.SilkS) (width 0.7))
+    (fp_line (start -7.366 -4.064) (end -7.366 4.318) (layer B.SilkS) (width 0.7))
+    (fp_line (start -7.366 4.318) (end 7.366 4.318) (layer B.SilkS) (width 0.7))
+    (fp_line (start 7.366 4.318) (end 7.366 -4.064) (layer B.SilkS) (width 0.7))
+    (fp_text user VCC (at -2.54 -2.794 unlocked) (layer B.SilkS)
+      (effects (font (size 0.75 0.75) (thickness 0.15)) (justify mirror))
+    )
+    (fp_text user SDA (at 0 -2.794 unlocked) (layer B.SilkS)
+      (effects (font (size 0.75 0.75) (thickness 0.15)) (justify mirror))
+    )
+    (fp_text user GPIO1 (at 3.937 -2.794 unlocked) (layer B.SilkS)
+      (effects (font (size 0.75 0.75) (thickness 0.15)) (justify mirror))
+    )
+    (fp_text user GND (at -2.54 3.048 unlocked) (layer B.SilkS)
+      (effects (font (size 0.75 0.75) (thickness 0.15)) (justify mirror))
+    )
+    (fp_text user SCL (at 0 3.048) (layer B.SilkS)
+      (effects (font (size 0.75 0.75) (thickness 0.15)) (justify mirror))
+    )
+    (fp_text user GPIO2 (at 3.937 3.048) (layer B.SilkS)
+      (effects (font (size 0.75 0.75) (thickness 0.15)) (justify mirror))
+    )
+    (pad 5 thru_hole circle (at 2.6 -1.25 270) (size 1.7272 1.7272) (drill 1.016) (layers *.Cu *.Mask)
+      (net 4 "Net-(X1-Pad5)"))
+    (pad 6 thru_hole circle (at 2.6 1.29 270) (size 1.7272 1.7272) (drill 1.016) (layers *.Cu *.Mask)
+      (net 5 "Net-(X1-Pad6)"))
+    (pad 3 thru_hole oval (at 0.06 -1.25 270) (size 1.7272 1.7272) (drill 1.016) (layers *.Cu *.Mask)
+      (net 6 "Net-(X1-Pad3)"))
+    (pad 4 thru_hole oval (at 0.06 1.29 270) (size 1.7272 1.7272) (drill 1.016) (layers *.Cu *.Mask)
+      (net 7 "Net-(X1-Pad4)"))
+    (pad 1 thru_hole oval (at -2.48 -1.25 270) (size 1.7272 1.7272) (drill 1.016) (layers *.Cu *.Mask)
+      (net 2 /VDD))
+    (pad 2 thru_hole rect (at -2.48 1.29 270) (size 1.7272 1.7272) (drill 1.016) (layers *.Cu *.Mask)
+      (net 1 GND))
+    (model ${KISYS3DMOD}/Connector_IDC.3dshapes/IDC-Header_2x03_P2.54mm_Vertical.wrl
+      (offset (xyz -2.5 1.2 -1.6))
+      (scale (xyz 1 1 1))
+      (rotate (xyz 180 0 90))
+    )
   )
   (module LOGO (layer F.Cu)
@@
     )
   )
-  (module my-ki-cad-parts:Badgelife-SAOv169-SAO-2x3 (layer F.Cu)
-    (at 1.4224 29.6164)
-    (descr "Through hole straight IDC box header, 2x03, 2.54mm pitch, double rows")
-    (tags "Through hole IDC box header THT 2x03 2.54mm double row")
-    (fp_text reference X1 (at 0 -5.842) (layer B.SilkS)
-      (effects (font (size 1 1) (thickness 0.15)) (justify mirror))
-    )
-    (fp_text value Badgelife_sao_connector_v169bis (at 0 -7.7) (layer F.Fab)
-      (effects (font (size 1 1) (thickness 0.15)))
-    )
-    (fp_text user %R (at 0.06 0.02 270) (layer F.Fab)
-      (effects (font (size 1 1) (thickness 0.15)))
-    )
-    (fp_line (start -2.54 -4.064) (end -7.366 -4.064) (layer B.SilkS) (width 0.7))
-    (fp_line (start 7.27964 -4.1148) (end 2.54 -4.1148) (layer B.SilkS) (width 0.7))
-    (fp_line (start -7.366 -4.064) (end -7.366 4.318) (layer B.SilkS) (width 0.7))
-    (fp_line (start -7.366 4.318) (end 7.366 4.318) (layer B.SilkS) (width 0.7))
-    (fp_line (start 7.366 4.318) (end 7.366 -4.064) (layer B.SilkS) (width 0.7))
-    (fp_text user VCC (at -2.54 -2.794 unlocked) (layer B.SilkS)
-      (effects (font (size 0.75 0.75) (thickness 0.15)) (justify mirror))
-    )
-    (fp_text user SDA (at 0 -2.794 unlocked) (layer B.SilkS)
-      (effects (font (size 0.75 0.75) (thickness 0.15)) (justify mirror))
-    )
-    (fp_text user GPIO1 (at 3.937 -2.794 unlocked) (layer B.SilkS)
-      (effects (font (size 0.75 0.75) (thickness 0.15)) (justify mirror))
-    )
-    (fp_text user GND (at -2.54 3.048 unlocked) (layer B.SilkS)
-      (effects (font (size 0.75 0.75) (thickness 0.15)) (justify mirror))
-    )
-    (fp_text user SCL (at 0 3.048) (layer B.SilkS)
-      (effects (font (size 0.75 0.75) (thickness 0.15)) (justify mirror))
-    )
-    (fp_text user GPIO2 (at 3.937 3.048) (layer B.SilkS)
-      (effects (font (size 0.75 0.75) (thickness 0.15)) (justify mirror))
-    )
-    (fp_circle (center -4.953 -3.429) (end -3.953 -3.429) (layer F.SilkS) (width 0.5))
-    (pad 5 thru_hole circle (at 2.6 -1.25 270) (size 1.7272 1.7272) (drill 1.016) (layers *.Cu *.Mask)
-      (net 4 "Net-(X1-Pad5)"))
-    (pad 6 thru_hole circle (at 2.6 1.29 270) (size 1.7272 1.7272) (drill 1.016) (layers *.Cu *.Mask)
-      (net 5 "Net-(X1-Pad6)"))
-    (pad 3 thru_hole oval (at 0.06 -1.25 270) (size 1.7272 1.7272) (drill 1.016) (layers *.Cu *.Mask)
-      (net 6 "Net-(X1-Pad3)"))
-    (pad 4 thru_hole oval (at 0.06 1.29 270) (size 1.7272 1.7272) (drill 1.016) (layers *.Cu *.Mask)
-      (net 7 "Net-(X1-Pad4)"))
-    (pad 1 thru_hole oval (at -2.48 -1.25 270) (size 1.7272 1.7272) (drill 1.016) (layers *.Cu *.Mask)
-      (net 2 /VDD))
-    (pad 2 thru_hole rect (at -2.48 1.29 270) (size 1.7272 1.7272) (drill 1.016) (layers *.Cu *.Mask)
-      (net 1 GND))
-    (model ${KISYS3DMOD}/Connector_IDC.3dshapes/IDC-Header_2x03_P2.54mm_Vertical.wrl
-      (offset (xyz -2.5 1.2 -1.6))
-      (scale (xyz 1 1 1))
-      (rotate (xyz 180 0 90))
-    )
-  )
